File: pcb/micromaus/maus.sch (EAGLE design)
At the start: 8 parts, among them IC1 EPF10K30-Q240, U1 ESP32-S2-WROOM

Commit message: feat: connector in sensor diagram
Parts:
- removed IC1: EPF10K30-Q240, altera:EPF10K30-Q240
- added C3, C4: 100nF, rcl:C-EUC0805
- added C5: 4.7uF, rcl:C-EUC0805
- added C6, C7: 10uF, rcl:C-EUC0805
- added CR1: L298P, shared:L298P
- added MOSFET2: SSM3J117TU(TE85L), SSM3J117TU:SSM3J117TU(TE85L)
- added PAD1, PAD2, PAD3, PAD4, PAD5, PAD6, PAD7, PAD8, PAD9: (no value), wirepad:1,6/0,8
- added Q1, Q2: BC817, BC817:BC817
- added R2, R3, R4: 10k, rcl:R-EU_R0805
- added SV1, SV2: (no value), con-harting-ml:ML6
- added U2: CH340C, CH340C:CH340C
- added U3: CP2102, CP2102:CP2102
- added U4: ESP32-S2-WROOM, ESP32-S2-WROOM:ESP32-S2-WROOM
- C1: value 4.7uF -> 10uF
Connections:
- new net AC_SENSOR1: PAD1.P
- new net AC_SENSOR3: PAD7.P
- new net AC_SESOR2: PAD4.P
- new net DTR: Q2.E, R3.1, U2.!DTR, U3.DTR
- new net ESP32_EN: Q1.C
- new net ESP32_IO0: Q2.C
- new net ESP32_RX: U2.TXD, U3.TXD
- new net ESP32_TX: U2.RXD, U3.RXD
- new net GND: C1.1, C6.1, C7.1, PAD2.P, PAD5.P, PAD8.P
- new net N$10: CR1.OUT2, U4.IO14
- new net N$11: CR1.INPUT1, U4.IO13
- new net N$12: CR1.INPUT2, U4.IO12
- new net N$13: CR1.VSS, SV1.4
- new net N$14: CR1.GND, SV1.3
- new net N$15: CR1.OUT3, SV1.6
- new net N$16: CR1.OUT4, SV1.5
- new net N$17: CR1.INPUT4, SV1.2
- new net N$18: CR1.INPUT3, SV1.1
- new net N$19: CR1.GND_3, SV2.3
- new net N$2: C3.1, U2.V3
- new net N$20: CR1.VS, SV2.4
- new net N$3: R2.2, U3.!SUSPEND
- new net N$5: Q1.B, R3.2
- new net N$7: C1.2, C6.2, C7.2, MOSFET2.3, PAD3.P, PAD6.P, PAD9.P
- new net N$8: CR1.GND_2, U4.GND
- new net N$9: CR1.OUT1, U4.IO15
- new net RTS: Q1.E, R4.1, U2.!RTS, U3.RTS
- new net SENSORS_ON/OF: MOSFET2.1
- new net USB_5V0: C2.1, C5.1, D1.2, U$1.VCC, U$2.A, U2.VCC, U3.REGIN, U3.VBUS
- new net VCC: MOSFET2.2
- net 0: now also C3.2, C4.2, C5.2, D1.1, R2.1, U2.GND, U3.GND; no longer C1.2
- net D+: now also D1.4, U2.UD+, U3.D+
- net D-: now also U2.UD-, U3.D-
- net N$4: now also C4.1, U3.VDD; no longer C1.1, C2.1, D1.2, D1.4, U$1.VCC, U$2.A
- net N$6: now also Q2.B, R4.2; no longer D1.1
