File: pcb/micromaus/maus.sch (EAGLE design)
At the start: 27 parts, among them IC1 AD712R, Q1 BSL307SP, T1 BC847, T2 BC847, U1 LP3965EMP-3.3

Commit message: Revert "Sensor_akt"
This reverts commit 3d197c96604575253fd7abde520af91cfe0fb7dc, reversing
changes made to 6c7812dcfceef42d4864bf92aec908c2e8f5b5d9.
Parts:
- removed C8: 6.8n, rcl:C-EUC0603
- removed IC1: AD712R, analog-devices:AD712R
- removed L1: 2.2u, rcl:L-EUPIS2816
- removed R1: (no value), rcl:R-EU_R0603
- removed R10, R11, R9: 22k, rcl:R-EU_R0603
- removed R12: 400k, rcl:R-EU_R0603
- removed R5: 10k, rcl:R-EU_R0603
- removed R6: 40.2k, rcl:R-EU_R0603
- removed R7: 7.68k, rcl:R-EU_R0603
- removed R8: 20, rcl:R-EU_R0603
- removed T1, T2: BC847, transistor:BC847
- added CR1: L298P, shared:L298P
- added D1: SP0503BAHTG, SP0503BAHTG:SP0503BAHTG
- added JP1: (no value), pinhead:PINHD-1X3
- added MOSFET2: SSM3J117TU(TE85L), SSM3J117TU:SSM3J117TU(TE85L)
- added PAD4, PAD5, PAD6, PAD7, PAD8, PAD9: (no value), wirepad:1,6/0,8
- added Q2: BC817, BC817:BC817
- added SV1, SV2: (no value), con-harting-ml:ML6
- added U$2: 1N5819, 1N5819:1N5819
- added U2: CH340C, CH340C:CH340C
- added U3: CP2102, CP2102:CP2102
- added U4: ESP32-S2-WROOM, ESP32-S2-WROOM:ESP32-S2-WROOM
- C1: value 22u -> 10uF; device rcl:C-EUC0603 -> rcl:C-EUC0805
- C2: value (none) -> 100nF; device rcl:C-EUC0603 -> rcl:C-EUC0805
- C3, C4: value 22u -> 100nF
- C5: value 22u -> 4.7uF
- C6: value 1u -> 10uF
- C7: value 1n -> 10uF; device rcl:C-EUC0603 -> rcl:C-EUC0805
- Q1: value BSL307SP -> BC817; device transistor-fet:BSL307SP -> BC817:BC817
- R2: value (none) -> 10k; device rcl:R-EU_R0603 -> rcl:R-EU_R0805
- R3: value 22k -> 10k; device rcl:R-EU_R0603 -> rcl:R-EU_R0805
- R4: value 100k -> 10k; device rcl:R-EU_R0603 -> rcl:R-EU_R0805
- U$1: value MP2333HSOT583 -> MICRO-USBV2; device MP2333H:MP2333HSOT583 -> microusb:MICRO-USBV2
- U1: value LP3965EMP-3.3 -> ESP32-S2-WROOM; device LP3965EMP-3.3:LP3965EMP-3.3 -> ESP32-S2-WROOM:ESP32-S2-WROOM
Connections:
- removed net +3V3: C2.1, IC1A.IN-, U1.SENSE/ADJ, U1.VOUT
- removed net +5V: C1.1, C4.1, C5.1, IC1P.V+, L1.2, Q1.S, R6.2, T1.C, T2.C, U1.VIN
- removed net BOOST_EN: R4.2, U$1.EN
- removed net EN_3V3: R9.2, T1.E, T2.E, U1.~SD
- removed net PGOOD: C7.1, R10.2, R3.1, U$1.PG
- removed net USB_VBUS: Q1.D, R11.1
- removed net VBAT: C3.1, R1.2, R12.1, R3.2, U$1.IN
- removed net VBUS_EN: IC1A.OUT, Q1.G, R12.2, R4.1
- new net 0: C2.2, C3.2, C4.2, C5.2, D1.1, R2.1, U$1.GND, U2.GND, U3.GND
- new net AC_SENSOR1: JP1.1
- new net AC_SENSOR3: PAD7.P
- new net AC_SESOR2: PAD4.P
- new net D+: D1.4, U$1.D+, U2.UD+, U3.D+
- new net D-: D1.3, U$1.D-, U2.UD-, U3.D-
- new net DTR: Q2.E, R3.1, U2.!DTR, U3.DTR
- new net ESP32_EN: Q1.C
- new net ESP32_IO0: Q2.C
- new net ESP32_RX: U1.RXD0, U2.TXD, U3.TXD
- new net ESP32_TX: U2.RXD, U3.RXD
- new net N$14: CR1.GND, SV1.3
- new net N$15: CR1.OUT3, SV1.6
- new net N$16: CR1.OUT4, SV1.5
- new net N$17: CR1.INPUT4, SV1.2
- new net N$18: CR1.INPUT3, SV1.1
- new net N$19: CR1.GND_3, SV2.3
- new net N$20: CR1.VS, SV2.4
- new net N$3: R2.2, U3.!SUSPEND
- new net N$4: C4.1, U3.VDD
- new net N$6: Q2.B, R4.2
- new net RTS: Q1.E, R4.1, U2.!RTS, U3.RTS
- new net SENSORS_ON/OF: MOSFET2.1
- new net USB_5V0: C2.1, C5.1, D1.2, U$1.VCC, U$2.A, U2.VCC, U3.REGIN, U3.VBUS
- new net VCC: MOSFET2.2
- net GND: now also C1.1, C6.1, C7.1, JP1.2, PAD5.P, PAD8.P; no longer C1.2, C2.2, C3.2, C4.2, C5.2, C7.2, C8.2, IC1P.V-, R2.1, R7.1, R9.1, U$1.GND, U1.GND
- net N$10: now also CR1.OUT2, U4.IO14; no longer C6.1, R8.1
- net N$11: now also CR1.INPUT1, U4.IO13; no longer C8.1, U$1.SS
- net N$12: now also CR1.INPUT2, U4.IO12; no longer R10.1, T2.B
- net N$13: now also CR1.VSS, SV1.4; no longer R11.2, T1.B
- net N$2: now also C3.1, U2.V3; no longer IC1A.IN+, R1.1, R2.2
- net N$5: now also Q1.B, R3.2; no longer C6.2, L1.1, U$1.SW
- net N$7: now also C1.2, C6.2, C7.2, JP1.3, MOSFET2.3, PAD6.P, PAD9.P; no longer R5.2, R6.1, R7.2
- net N$8: now also CR1.GND_2, U4.GND; no longer R5.1, U$1.FB
- net N$9: now also CR1.OUT1, U4.IO15; no longer R8.2, U$1.BST
Other:
- note removed: "Die widerstandswerte hier sind noch zu durchdenken, es gibt einen maximalstrom für BOOST_EN. idee ist: beim hochfahren von Batterie ist VBUS_EN erst mal undefiniert und wird nicht getrieben (hoffentlich) weil der komparator keinen Strom bekommt. dann zieht VBAT das hoch."
- note removed: "alternativ EN des MP2333H an den ausgang des opamp? muss dann der AD712R an VBAT betrieben werden?"
- note removed: "alternativ dioden-or?"
- note removed: "muss das ein depletion type sein?"
- note removed: "todo widerstandswerte"
