File: pcb/maus_backup.brd (EAGLE design)
At the start: 100 x 101 mm, 79 parts, among them IC1 AP1509-50SG-13, J1 SS-52300-001, Q2 BSS123, Q3 BSS123, Q4 BSS123, Q6 PMN30XPEA, Q7 PMN30XPEA, U1 ESP32-S2-WROOM, U2 CH340C, U4 LP3965EMP-3.3, U6 LM358DR

Commit message: fuck my life 2.0
Routing:
- net H_EN_A: track 69.9 -> 7.74 mm, vias 4 -> 0
- net ESP32_M1_1: track 71.2 -> 11.9 mm, vias 4 -> 0
- net ESP32_M1_2: track 60.6 -> 6.27 mm, vias 4 -> 0
- net VBAT: track 131.0 -> 105.7 mm, vias 5 -> 3
- net ESP32_M2_2: track 39.7 -> 16.6 mm
- net M2_M+: track 36.8 -> 15.7 mm, vias 2 -> 0
- net H_EN_B: track 44.3 -> 28.1 mm
- net M2_M-: track 48.8 -> 34.9 mm, vias 2 -> 0
